File: kicad/rev6/amigahid-pico-rev6.kicad_sch (KiCad schematic)
At the start: 58 parts, among them J1 Amiga Keyboard, J2 Debug/programming, J3 i2c header, J4 USB_A, J5 Controller 1, J6 Controller 2, Q1 BSS138, Q10 BSS138, Q11 BSS138, Q12 BSS138, Q13 BSS138, Q14 BSS138, Q15 BSS138, Q16 BSS138, Q17 BSS138, Q2 BSS138, Q3 BSS138, Q4 BSS138, Q5 BSS138, Q6 BSS138, Q7 BSS138, Q8 BSS138, Q9 BSS138, U1 Pico

Commit message: kicad: rev6 schematic
Replace the rev5 schematic the rev6 project was bootstrapped from with the
rev6 design. Flat single sheet (A1), wired by net labels in the rev5 style;
every no-connect carries an explicit flag. ERC reports 0 errors and 0
warnings; tools/check_rev6_netlist.py passes all 349 assertions against
src/config.h and the rev6 connectivity spec.

Gone from rev5: the J5/J6 IDC controller headers, the single unprotected +5V
node, the IDC interleave compensation, and the 17-channel shifter bank.

Power tree. AMIGA_5V (J1.4 || J9.5 || J10.4) -> F1 750 mA polyfuse -> D1
SS34 -> SYS5V; the USB-C aux input feeds SYS5V through D2. SYS5V drives the
module's VSYS (pin 39, not VBUS, so the module's own MBR120 diode-ORs PC USB
power while installed), the 19 high-side pull-ups, F2 (500 mA) -> USBA_5V
and F3 (200 mA) -> KBIN_5V. Bulk 220uF + 10uF + 100nF on SYS5V, 220uF +
100nF on USBA_5V. +3V3 has exactly one source: the module's pin 36.

Level shifting. 19 discrete BSS138 channels, gate on +3V3, source on the
3V3-side net with a 10k pull-up to +3V3, drain on the 5V-side net with a 10k
pull-up to SYS5V: 3 keyboard-out, 2 keyboard-in, 7 + 7 controller port.

Connectors. J1/J8 A500-style 1x8 keyboard headers out and in with the reset
line wire-ORed in copper and the power/drive LED pins passed through; J9/J11
DIN5 and J10/J12 mini-DIN6 sockets paralleled onto the same two groups;
P1/P2 DE9 male controller ports; J2 debug (UART + SWD off the module's
mid-board pads); J3 OLED with the 4.7k I2C pull-ups rev5 lacked; J7 spare
GP28 header; JP1 solder jumper (open) strapping the keyboard-in power LED
pin to SYS5V for standalone use.

Protection. USBLC6-2SC6 on the USB-A data pair and VBUS, and a ground-clamp
PESD-class TVS on each of the 19 Amiga-facing 5V lines. No rail-steering
arrays anywhere: they would phantom-power SYS5V from Amiga-driven lines with
the board unpowered.

LCSC codes are carried in the symbols for JLC assembly. Polyfuses, bulk
electrolytics and the TVS c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
Parts:
- removed J5: Controller 1, Connector_IDC:IDC-Header_2x05_P2.54mm_Vertical, symbol Connector_Generic:Conn_02x05_Odd_Even
- removed J6: Controller 2, Connector_IDC:IDC-Header_2x05_P2.54mm_Vertical, symbol Connector_Generic:Conn_02x05_Odd_Even
- removed U1: Pico, MCU_RaspberryPi_and_Boards:RPi_Pico_SMD_TH, symbol MCU_RaspberryPi_and_Boards:Pico
- added C1, C4: 220uF, Capacitor_SMD:CP_Elec_6.3x7.7, symbol Device:C
- added C2: 10uF, Capacitor_SMD:C_0805_2012Metric, symbol Device:C
- added C3, C5: 100nF, Capacitor_SMD:C_0603_1608Metric, symbol Device:C
- added D1, D2: SS34, Diode_SMD:D_SMA, symbol Device:D_Schottky
- added D10, D11, D12, D13, D14, D15, D16, D17, D18, D19, D20, D21, D22, D23, D24, D25, D26, D27, D28: PESD5V0S1BA, Diode_SMD:D_SOD-523, symbol Device:D_TVS
- added F1: 750mA, Fuse:Fuse_1812_4532Metric, symbol Device:Polyfuse
- added F2: 500mA, Fuse:Fuse_1812_4532Metric, symbol Device:Polyfuse
- added F3: 200mA, Fuse:Fuse_1812_4532Metric, symbol Device:Polyfuse
- added J10: PS/2 KBD OUT, rev6:MiniDIN6_PS2_Socket_CUI_MD-60S, symbol rev6:MiniDIN6_PS2_Socket
- added J11: DIN5 KBD IN, rev6:DIN5_180deg_Socket_Kycon_KCDX-5S-N, symbol rev6:DIN5_180deg_Socket
- added J12: PS/2 KBD IN, rev6:MiniDIN6_PS2_Socket_CUI_MD-60S, symbol rev6:MiniDIN6_PS2_Socket
- added J13: USB-C AUX 5V, Connector_USB:USB_C_Receptacle_GCT_USB4135-GF-A_6P_TopMnt_Horizontal, symbol Connector:USB_C_Receptacle_PowerOnly_6P
- added J7: SPARE GP28, Connector_PinHeader_2.54mm:PinHeader_1x03_P2.54mm_Vertical, symbol Connector_Generic:Conn_01x03
- added J8: A500 KBD IN, Connector_PinHeader_2.54mm:PinHeader_1x08_P2.54mm_Vertical, symbol Connector_Generic:Conn_01x08
- added J9: DIN5 KBD OUT, rev6:DIN5_180deg_Socket_Kycon_KCDX-5S-N, symbol rev6:DIN5_180deg_Socket
- added JP1: KBIN PWRLED, Jumper:SolderJumper-2_P1.3mm_Open_RoundedPad1.0x1.5mm, symbol Jumper:SolderJumper_2_Open
- added LED1: red, LED_SMD:LED_0603_1608Metric, symbol Device:LED
- added LED2: green, LED_SMD:LED_0603_1608Metric, symbol Device:LED
- added P1: DE9 MALE PORT 1, Connector_Dsub:DSUB-9_Pins_Horizontal_P2.77x2.84mm_EdgePinOffset4.94mm_Housed_MountingHolesOffset4.94mm, symbol Connector:DE9_Pins_MountingHoles
- added P2: DE9 MALE PORT 2, Connector_Dsub:DSUB-9_Pins_Horizontal_P2.77x2.84mm_EdgePinOffset4.94mm_Housed_MountingHolesOffset4.94mm, symbol Connector:DE9_Pins_MountingHoles
- added Q18, Q19: BSS138, Package_TO_SOT_SMD:SOT-23, symbol Transistor_FET:BSS138
- added R35, R36, R37, R38: 10k, Resistor_SMD:R_0603_1608Metric, symbol Device:R
- added R39, R40: 1k, Resistor_SMD:R_0603_1608Metric, symbol Device:R
- added R41, R42: 4.7k, Resistor_SMD:R_0603_1608Metric, symbol Device:R
- added R43, R44: 5.1k, Resistor_SMD:R_0603_1608Metric, symbol Device:R
- added U1: PicoW, rev6:RPi_PicoW_SMD_TH, symbol rev6:PicoW
- added U2: USBLC6-2SC6, Package_TO_SOT_SMD:SOT-23-6, symbol Power_Protection:USBLC6-2SC6
- J1: value Amiga Keyboard -> A500 KBD OUT
- J2: value Debug/programming -> DEBUG UART+SWD; footprint Connector_PinHeader_2.54mm:PinHeader_1x06_P2.54mm_Horizontal -> Connector_PinHeader_2.54mm:PinHeader_1x06_P2.54mm_Vertical
- J3: value i2c header -> OLED I2C
- J4: value USB_A -> USB-A HOST
- Q1, Q10, Q11, Q12, Q13, Q14, Q15, Q16, Q17, Q2, Q3, Q4, Q5, Q6, Q7, Q8, Q9: LCSC (none) -> C82227
- R1, R10, R11, R12, R13, R14, R15, R16, R17, R18, R19, R2, R20, R21, R22, R23, R24, R25, R26, R27, R28, R29, R3, R30, R31, R32, R33, R34, R4, R5, R6, R7, R8, R9: value R1002 -> 10k; LCSC (none) -> C25804
Connections:
- net +3V3: now also R1.1, R11.1, R13.1, R15.1, R17.1, R19.1, R21.1, R23.1, R25.1, R27.1, R29.1, R3.1, R31.1, R33.1, R5.1, R7.1, R9.1, J7.2 (Pin_2), Q18.1 (G), Q19.1 (G), R35.1, R37.1, R41.1, R42.1, U1.36 (3V3); no longer R10.2, R12.2, R14.2, R16.2, R18.2, R2.2, R20.2, R22.2, R24.2, R26.2, R28.2, R30.2, R32.2, R34.2, R4.2, R6.2, R8.2
- net GND: now also J4.SH (Shield), C1.2, C2.2, C3.2, C4.2, C5.2, D10.2 (A2), D11.2 (A2), D12.2 (A2), D13.2 (A2), D14.2 (A2), D15.2 (A2), D16.2 (A2), D17.2 (A2), D18.2 (A2), D19.2 (A2), D20.2 (A2), D21.2 (A2), D22.2 (A2), D23.2 (A2), D24.2 (A2), D25.2 (A2), D26.2 (A2), D27.2 (A2), D28.2 (A2), J10.3, J10.SH (SHIELD), J11.4, J11.MP, J12.3, J12.SH (SHIELD), J13.A12 (GND), J13.B12 (GND), J13.SH (SHIELD), J7.3 (Pin_3), J8.6 (Pin_6), J9.4, J9.MP, LED1.1 (K), LED2.1 (K), P1.8, P1.SH (PAD), P2.8, P2.SH (PAD), R43.2, R44.2, U1.13 (GND), U1.18 (GND), U1.23 (GND), U1.28 (GND), U1.3 (GND), U1.33 (AGND), U1.38 (GND), U1.42 (GND), U1.8 (GND), U1.SH (SHIELD), U2.2 (GND); no longer J4.5 (Shield)
- net kbclock: now also Q3.3 (D), R6.2, D12.1 (A1), J10.5, J9.1; no longer Q1.3 (D), R1.1
- net kbdata: now also R4.2, D11.1 (A1), J10.1, J9.2; no longer R3.1
- net kbreset: now also Q1.3 (D), R2.2, D10.1 (A1), J8.3 (Pin_3); no longer Q3.3 (D), R5.1
- net swclk: now also U1.41 (SWCLK)
- net swdio: now also U1.43 (SWDIO)
- removed net +5V: J1.4 (Pin_4), J4.1 (VBUS), R1.2, R11.2, R13.2, R15.2, R17.2, R19.2, R21.2, R23.2, R25.2, R27.2, R29.2, R3.2, R31.2, R33.2, R5.2, R7.2, R9.2
- net cont1 b1 renamed cont1_b1
- net cont1_b1: now also R16.2, D17.1 (A1), P1.6; no longer R15.1
- net cont1 b2 renamed cont1_b2
- net cont1_b2: now also R18.2, D18.1 (A1), P1.9; no longer R17.1
- net cont1 b3 renamed cont1_b3
- net cont1_b3: now also R20.2, D19.1 (A1), P1.5; no longer R19.1
- net cont1 h renamed cont1_h
- net cont1_h: now also R12.2, D15.1 (A1), P1.2; no longer R11.1
- net cont1 hq renamed cont1_hq
- net cont1_hq: now also R8.2, D13.1 (A1), P1.4; no longer R7.1
- net cont1 v renamed cont1_v
- net cont1_v: now also R14.2, D16.1 (A1), P1.1; no longer R13.1
- net cont1 vq renamed cont1_vq
- net cont1_vq: now also R10.2, D14.1 (A1), P1.3; no longer R9.1
- net cont2 b1 renamed cont2_b1
- net cont2_b1: now also R30.2, D24.1 (A1), P2.6; no longer R29.1
- net cont2 b2 renamed cont2_hq
- net cont2_hq: now also R32.2, D25.1 (A1), P2.4; no longer R31.1
- net cont2 b3 renamed cont2_vq
- net cont2_vq: now also R34.2, D26.1 (A1), P2.3; no longer R33.1
- net cont2 h renamed kbin_dat
- net kbin_dat: now also R24.2, D21.1 (A1), J11.2, J12.1, J8.2 (Pin_2); no longer R23.1
- net cont2 hq renamed cont2_b2
- net cont2_b2: now also R28.2, D23.1 (A1), P2.9; no longer R27.1
- net cont2 v renamed kbin_clk
- net kbin_clk: now also R22.2, D20.1 (A1), J11.1, J12.5, J8.1 (Pin_1); no longer R21.1
- net cont2 vq renamed cont2_b3
- net cont2_b3: now also R26.2, D22.1 (A1), P2.5; no longer R25.1
- net i2c scl renamed i2c_scl
- net i2c_scl: now also R42.2, U1.5 (GPIO3)
- net i2c sda renamed i2c_sda
- net i2c_sda: now also R41.2, U1.4 (GPIO2)
- net kbdriveled renamed kb_drvled
- net kb_drvled: now also J8.8 (Pin_8)
- net kbpowerled renamed kb_pwrled
- net kb_pwrled: now also J8.7 (Pin_7), JP1.1 (A)
- net lcont1 b1 renamed SYS5V
- net SYS5V: now also R10.1, R12.1, R14.1, R18.1, R2.1, R20.1, R22.1, R24.1, R26.1, R28.1, R30.1, R32.1, R34.1, R4.1, R6.1, R8.1, C1.1, C2.1, C3.1, D1.1 (K), D2.1 (K), F2.1, F3.1, JP1.2 (B), R36.1, R38.1, U1.39 (VSYS); no longer Q8.2 (S)
- net lcont1 b2 renamed cont1_b2_lo
- net cont1_b2_lo: now also R17.2, U1.16 (GPIO12); no longer R18.1
- net lcont1 b3 renamed cont1_b3_lo
- net cont1_b3_lo: now also R19.2, U1.17 (GPIO13); no longer R20.1
- net lcont1 h renamed cont1_h_lo
- net cont1_h_lo: now also R11.2, U1.12 (GPIO9); no longer R12.1
- net lcont1 hq renamed cont1_hq_lo
- net cont1_hq_lo: now also R7.2, U1.10 (GPIO7); no longer R8.1
- net lcont1 v renamed cont1_v_lo
- net cont1_v_lo: now also R13.2, U1.14 (GPIO10); no longer R14.1
- net lcont1 vq renamed cont1_vq_lo
- net cont1_vq_lo: now also R9.2, U1.11 (GPIO8); no longer R10.1
- net lcont2 b1 renamed cont2_b1_lo
- net cont2_b1_lo: now also R29.2, U1.26 (GPIO20); no longer R30.1
- net lcont2 b2 renamed cont2_hq_lo
- net cont2_hq_lo: now also R31.2, U1.27 (GPIO21); no longer R32.1
- net lcont2 b3 renamed cont2_vq_lo
- net cont2_vq_lo: now also R33.2, U1.29 (GPIO22); no longer R34.1
- net lcont2 h renamed kbin_dat_lo
- net kbin_dat_lo: now also R23.2, U1.20 (GPIO15); no longer R24.1
- net lcont2 hq renamed cont2_b2_lo
- net cont2_b2_lo: now also R27.2, U1.25 (GPIO19); no longer R28.1
- net lcont2 v renamed kbin_clk_lo
- net kbin_clk_lo: now also R21.2, U1.19 (GPIO14); no longer R22.1
- net lcont2 vq renamed cont2_b3_lo
- net cont2_b3_lo: now also R25.2, U1.24 (GPIO18); no longer R26.1
- net lkbclock renamed kbreset_lo
- net kbreset_lo: now also R1.2, U1.6 (GPIO4); no longer R2.1
- net lkbdata renamed kbdata_lo
- net kbdata_lo: now also R3.2, U1.7 (GPIO5); no longer R4.1
- net lkbreset renamed kbclock_lo
- net kbclock_lo: now also R5.2, U1.9 (GPIO6); no longer R6.1
- net uart rx renamed uart_rx
- net uart_rx: now also U1.2 (GPIO1)
- net uart tx renamed uart_tx
- net uart_tx: now also U1.1 (GPIO0)
- net usb d+ renamed usb_dp
- net usb_dp: now also U1.TP3, U2.3 (I/O2), U2.4 (I/O2)
- net usb d- renamed usb_dm
- net usb_dm: now also U1.TP2, U2.1 (I/O1), U2.6 (I/O1)
- new net AMIGA_5V: F1.1, J1.4 (Pin_4), J10.4, J9.5
- new net AMIGA_5V_FUSED: D1.2 (A), F1.2
- new net AUX_5V: D2.2 (A), J13.A9 (VBUS), J13.B9 (VBUS)
- new net KBIN_5V: F3.2, J11.5, J12.4, J8.4 (Pin_4)
- new net USBA_5V: C4.1, C5.1, F2.2, J4.1 (VBUS), U2.5 (VBUS)
- new net cont1_b1_lo: Q8.2 (S), R15.2, U1.15 (GPIO11)
- new net cont2_h: D27.1 (A1), P2.2, Q18.3 (D), R36.2
- new net cont2_h_lo: Q18.2 (S), R35.2, U1.31 (GPIO26_ADC0)
- new net cont2_v: D28.1 (A1), P2.1, Q19.3 (D), R38.2
- new net cont2_v_lo: Q19.2 (S), R37.2, U1.32 (GPIO27_ADC1)
- new net gp28: J7.1 (Pin_1), U1.34 (GPIO28_ADC2)
- new net led1_a: LED1.2 (A), R39.2
- new net led1_drv: R39.1, U1.21 (GPIO16)
- new net led2_a: LED2.2 (A), R40.2
- new net led2_drv: R40.1, U1.22 (GPIO17)
- new net usb_cc1: J13.A5 (CC1), R43.1
- new net usb_cc2: J13.B5 (CC2), R44.1
Other:
- note added: "DE9s are male: use straight-through F-F cables, NOT null-modem."
- note added: "F1 sizing is provisional - confirm on the bench before fab (M5)."
- note added: "LCSC codes marked TBD: polyfuses, bulk electrolytics and the TVS clamps are sourced at fab time (M4)."
- note added: "Warning: the three OUT connectors share AMIGA_5V pre-fuse - connect ONE amiga at a time."
- note added: "bss138 level shift channels - 3v3 low side / sys5v high side"
- note added: "controller ports (de9 male, straight-through f-f cables)"
- note added: "debug / display / spare / status"
- note added: "esd clamps - amiga facing lines, ground clamp only"
- note added: "from real amiga keyboard"
- note added: "mcu - raspberry pi pico w / pico 2 w"
- note added: "power tree"
- note added: "to amiga (connect one machine at a time)"
- note added: "usb host + aux 5v input"
- note removed: "Amiga controller port (D-Sub 9, socket at peripheral side) pin m j 1 V UP 2 H DN 3 VQ LF 4 HQ RT 5 b3 b3 6 b1 b1 7 +5V +5V 8 GND GND 9 b2 b2 (n.b. idc ports are interleaved; d-subs are numbered top row, bottom row)"
- note removed: "Controller 1 level conversion"
- note removed: "Controller 2 level conversion"
- note removed: "I/O Ports"
- note removed: "Keyboard level conversion"
- note removed: "MCU Section"

Commit message: kicad: fix rev6 part numbers, packages and power tree
Part numbers, all verified against the vendor/LCSC listing:

- Q1-Q19 carried LCSC C82227, which is a TI HDC1080 humidity sensor in
  WSON-6, not a BSS138. Nineteen parts - the largest assembly line item -
  would have been rejected or populated wrong. Now C78284 (JSCJ BSS138,
  SOT-23).
- D10-D28 paired the value PESD5V0S1BA with Diode_SMD:D_SOD-523. The -BA
  suffix is SOD-323 (1.7 x 1.25 mm body); it cannot sit on a SOD-523 land
  (pads at +-0.70 vs +-1.05). Footprint moved to D_SOD-323 and the LCSC
  placeholder replaced with the real stocked code C19224, which the plan
  wanted picked at this milestone anyway.
- LED2 carried C2297 = KT-0805G, an 0805 part on an 0603 land, and at Vf
  2.6-3.1 V an InGaN green cannot light from 3V3 through 1k (0.1-0.4 mA).
  Now C2289 / KT-0603YG, genuinely 0603 and Vf 2.0-2.2 V, which puts it
  at ~1.2 mA to match LED1's red.

Power tree:

- F3 (keyboard-IN rail) was MF-MSMF020-2: 200 mA hold against a serial
  Amiga keyboard's 100-150 mA, i.e. 50-75% of Ihold with R1max 6.0 ohm,
  so it self-heats, droops and can trip on cold start - which per the
  design leaves _KBRESET asserted. Now MF-MSMF050-2 (Rmin 0.15/R1max 1.0,
  same part as F2), and KBIN_5V gains local bulk (C6 10uF, C7 100nF); it
  previously had no decoupling at all.
- JP1 strapped kb_pwrled straight to SYS5V. The A500 carries the power
  LED's ballast on the motherboard side, so closing the jumper put the
  full rail across a bare LED, and leaving it closed with J1 cabled to a
  live A500 back-fed the machine's LED-drive node. R45 (470R) now sits in
  the JP1 leg, with a sheet note that JP1 is standalone-only.
- C4 drops 220uF -> 150uF. It sits behind F2 but is still charged from
  AMIGA_5V at plug-in, so the machine saw 440uF against the plan's
  <=220uF inrush budget; 150uF still clears the USB host requirement.
- C1/C4 are aluminium electrolytics on a polarised CP_Elec land but were
  drawn with the unpolari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
Parts:
- added C6: 10uF, Capacitor_SMD:C_0805_2012Metric, symbol Device:C
- added C7: 100nF, Capacitor_SMD:C_0603_1608Metric, symbol Device:C
- added D29, D30: PESD5V0S1BA, Diode_SMD:D_SOD-323, symbol Device:D_TVS
- added R45: 470, Resistor_SMD:R_0603_1608Metric, symbol Device:R
- C1: symbol Device:C -> Device:C_Polarized
- C4: value 220uF -> 150uF; symbol Device:C -> Device:C_Polarized; LCSC TBD:220uF/16V SMD alu -> TBD:150uF/16V SMD alu
- D10, D11, D12, D13, D14, D15, D16, D17, D18, D19, D20, D21, D22, D23, D24, D25, D26, D27, D28: footprint Diode_SMD:D_SOD-523 -> Diode_SMD:D_SOD-323; LCSC TBD:PESD5V0S1BA -> C19224
- F3: value 200mA -> 500mA; MPN MF-MSMF020-2 -> MF-MSMF050-2
- LED2: value green -> yellow-green; LCSC C2297 -> C2289; MPN (none) -> KT-0603YG
- Q1, Q10, Q11, Q12, Q13, Q14, Q15, Q16, Q17, Q18, Q19, Q2, Q3, Q4, Q5, Q6, Q7, Q8, Q9: LCSC C82227 -> C78284
Connections:
- net GND: now also C6.2, C7.2, D29.2 (A2), D30.2 (A2)
- net KBIN_5V: now also C6.1, C7.1
- net SYS5V: now also R45.2; no longer JP1.2 (B)
- net kb_drvled: now also D30.1 (A1)
- net kb_pwrled: now also D29.1 (A1)
- new net: JP1.2 (B), R45.1
Other:
- note added: "=> USB-A is rated for low-power HID here. A powered hub or the J13 aux 5V input is REQUIRED for high-current devices. D1 stays an SS34: the LM66100 ideal-diode option was weighed and declined; revisit if M5 measures worse."
- note added: "F1 is a PLACEHOLDER: measure full-stack current on the bench and re-size before fab (M4), not at bring-up. It must trip before any host-side fuse (A4000 keyboard port ~100 mA)."
- note added: "JP1 is for STANDALONE use only - no amiga cabled to J1. R45 limits the strap to ~5 mA; the A500 drives kb_pwrled from its own side."
- note added: "LCSC codes marked TBD: polyfuses and bulk electrolytics are sourced at fab time (M4). Everything else is pinned to a stocked part number."
- note added: "Series drop on amiga power: SYS5V = AMIGA_5V - F1 (0.11-0.45 ohm) - D1 (SS34, ~0.35 V) ~= 4.5 V. USBA_5V is another F2 down: ~4.4-4.6 V at HID loads, under 4.4 V approaching 500 mA."
- note added: "Verify J9/J11 (DIN5), J10/J12 (mini-DIN6) and P1/P2 (DE9, EdgePinOffset4.94mm) against physical samples before fab - connector variant mismatch is the classic re-spin cause."
- note removed: "F1 sizing is provisional - confirm on the bench before fab (M5)."
- note removed: "LCSC codes marked TBD: polyfuses, bulk electrolytics and the TVS clamps are sourced at fab time (M4)."

Commit message: kicad: fix rev6 placement ahead of routing
J4 was fitted back to front: the Molex 67643 land pattern mates at its
local +y, so the receptacle was pointing into the board and its pads sat
2.8 mm from the south edge instead of 13.5 mm.  Turned round and pushed
out, which also brings the USB tap within reach - usb_dp/usb_dm could not
have been routed under 25 mm the way it stood.

Other placement work:

  - U1 1 mm north, opening a component band between the module and J4;
    R7..R14 follow so the SWD pads keep clear of R9.
  - U2 (USBLC6) and F2 to the top side as the layout brief requires, U2
    turned 90 deg so each USB line runs straight down one pad column
    from the tap to the connector.  C4 follows.
  - TP2/TP3 declared castellated pads: they are half vias deliberately
    bisected by the milled USB-tap window, as on rev 5, and that is what
    the pad property is for.
  - antenna rule area grown to the full 11 x 15.8 mm guarded region and
    set to forbid footprints as well as copper.
  - silkscreen trimmed back inside the board outline (edge connectors
    were printing past it) and the labels that landed on J4/U2 moved.
  - the edited footprints are vendored into rev6.pretty so the board no
    longer differs from its libraries; U1's six unnamed editing groups
    are dropped, and the zone points FootprintSave writes are corrected
    (it rotates footprint rule areas into the library frame but does not
    translate them).
  - the JP1/R45 link gets a name, kb_pwrled_bal, so schematic parity has
    something to match.

DRC is clean bar the 291 unrouted connections; netlist checker 356/356.
Parts:
- J4: footprint Connector_USB:USB_A_Molex_67643_Horizontal -> rev6:USB_A_Molex_67643_Horizontal
- P1, P2: footprint Connector_Dsub:DSUB-9_Pins_Horizontal_P2.77x2.84mm_EdgePinOffset4.94mm_Housed_MountingHolesOffset4.94mm -> rev6:DSUB-9_Pins_Horizontal_P2.77x2.84mm_EdgePinOffset4.94mm_Housed_MountingHolesOffset4.94mm
Connections:
- net kb_pwrled_bal: now reaches JP1.2 (B), R45.1
Changed lines of the file:
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@@
 			)
 		)
-		(property "Footprint" "Connector_Dsub:DSUB-9_Pins_Horizontal_P2.77x2.84mm_EdgePinOffset4.94mm_Housed_MountingHolesOffset4.94mm"
+		(property "Footprint" "rev6:DSUB-9_Pins_Horizontal_P2.77x2.84mm_EdgePinOffset4.94mm_Housed_MountingHolesOffset4.94mm"
 			(at 74.93 434.34 0)
 			(hide yes)
@@
 			)
 		)
-		(property "Footprint" "Connector_Dsub:DSUB-9_Pins_Horizontal_P2.77x2.84mm_EdgePinOffset4.94mm_Housed_MountingHolesOffset4.94mm"
+		(property "Footprint" "rev6:DSUB-9_Pins_Horizontal_P2.77x2.84mm_EdgePinOffset4.94mm_Housed_MountingHolesOffset4.94mm"
 			(at 74.93 504.19 0)
 			(hide yes)
@@
 		)
 	)
+	(label "kb_pwrled_bal"
+		(at 400.05 168.91 0)
+		(effects
+			(font
+				(size 1.27 1.27)
+			)
+			(justify left bottom)
+		)
+	)
 	(label "kb_pwrled"
 		(at 381 168.91 180)
@@
 			)
 		)
-		(property "Footprint" "Connector_USB:USB_A_Molex_67643_Horizontal"
+		(property "Footprint" "rev6:USB_A_Molex_67643_Horizontal"
 			(at 320.04 424.18 0)
 			(hide yes)

Commit message: kicad: pin real part numbers across the rev6 bom
the last five TBD entries get real, in-stock lcsc codes: C1 220uF and C4
150uF become panasonic FK cans (C128533 / C413656) on the 6.3x7.7 land,
and the three polyfuses become the bourns MF-MSMF parts their MPN fields
already named (F1 750mA C84140, F2/F3 500mA C17313).

everything that is hand-soldered - all thirteen connectors, the pico w
module and the solder jumper - gets a Sourcing field instead of an lcsc
code, so jlc never sees them and nobody has to guess later. the DE9 line
is the one worth reading: the board's land is the 5.0 mm footprint, so
the common 0.318 in parts do not fit.

fields only, no connectivity touched. the pcb footprints carry copies of
these fields, so they are updated in step or schematic parity fails.
Parts:
- C1: LCSC TBD:220uF/16V SMD alu -> C128533; MPN (none) -> EEE-FK1C221XP
- C4: LCSC TBD:150uF/16V SMD alu -> C413656; MPN (none) -> EEE-FKC151XAP
- F1: LCSC TBD:MF-MSMF series -> C84140
- F2, F3: LCSC TBD:MF-MSMF series -> C17313
- J1, J8: Sourcing (none) -> generic 2.54 mm pin header, 1x8 vertical - hand-solder, not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
- J10, J12: Sourcing (none) -> Same Sky (CUI Devices) MD-60S (mini-DIN 6 socket, right-ang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
- J11, J9: Sourcing (none) -> Kycon KCDX-5S-N (DIN 41524 5-pin 180 deg socket, right-angl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
- J13: Sourcing (none) -> GCT USB4135-GF-A (USB-C 6P power-only receptacle, top-mount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
- J2: Sourcing (none) -> generic 2.54 mm pin header, 1x6 vertical - hand-solder, not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
- J3: Sourcing (none) -> generic 2.54 mm pin header, 1x4 vertical - hand-solder, not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
- J4: Sourcing (none) -> Molex 67643-3910 (USB-A receptacle, right-angle THT; 67643-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
- J7: Sourcing (none) -> generic 2.54 mm pin header, 1x3 vertical - hand-solder, not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
- JP1: Sourcing (none) -> none - solder bridge, no part to buy
- P1, P2: Sourcing (none) -> Power Dynamics PDI-09S-5 (DE9 male, right-angle THT, 5.0 mm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
- U1: Sourcing (none) -> Raspberry Pi Pico W or Pico 2 W module - hand-solder by cas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
Changed lines of the file:
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@@
 			)
 		)
+		(property "Sourcing" "Raspberry Pi Pico W or Pico 2 W module - hand-solder by castellations or fit on 2x20 sockets, not JLC-assembled"
+			(at 210.82 200.66 0)
+			(hide yes)
+			(effects
+				(font
+					(size 1.27 1.27)
+				)
+			)
+		)
 		(pin "1"
 		)
@@
 			)
 		)
+		(property "Sourcing" "generic 2.54 mm pin header, 1x8 vertical - hand-solder, not JLC-assembled"
+			(at 74.93 60.96 0)
+			(hide yes)
+			(effects
+				(font
+					(size 1.27 1.27)
+				)
+			)
+		)
 		(pin "1"
 		)
@@
 			)
 		)
+		(property "Sourcing" "Kycon KCDX-5S-N (DIN 41524 5-pin 180 deg socket, right-angle THT) - hand-solder, not JLC-assembled"
+			(at 74.93 121.92 0)
+			(hide yes)
+			(effects
+				(font
+					(size 1.27 1.27)
+				)
+			)
+		)
 		(pin "1"
 		)
@@
 			)
 		)
+		(property "Sourcing" "Same Sky (CUI Devices) MD-60S (mini-DIN 6 socket, right-angle THT; Kycon KMDGX-6S-N shares the grid) - hand-solder, not JLC-assembled"
+			(at 74.93 168.91 0)
+			(hide yes)
+			(effects
+				(font
+					(size 1.27 1.27)
+				)
+			)
+		)
 		(pin "1"
 		)
@@
 			)
 		)
+		(property "Sourcing" "generic 2.54 mm pin header, 1x8 vertical - hand-solder, not JLC-assembled"
+			(at 74.93 241.3 0)
+			(hide yes)
+			(effects
+				(font
+					(size 1.27 1.27)
+				)
+			)
+		)
 		(pin "1"
 		)
@@
 			)
 		)
+		(property "Sourcing" "Kycon KCDX-5S-N (DIN 41524 5-pin 180 deg socket, right-angle THT) - hand-solder, not JLC-assembled"
+			(at 74.93 302.26 0)
+			(hide yes)
+			(effects
+				(font
+					(size 1.27 1.27)
+				)
+			)
+		)
 		(pin "1"
 		)
@@
 			)
 		)
+		(property "Sourcing" "Same Sky (CUI Devices) MD-60S (mini-DIN 6 socket, right-angle THT; Kycon KMDGX-6S-N shares the grid) - hand-solder, not JLC-assembled"
+			(at 74.93 349.25 0)
+			(hide yes)
+			(effects
+				(font
+					(size 1.27 1.27)
+				)
+			)
+		)
 		(pin "1"
 		)
@@
 			)
 		)
+		(property "Sourcing" "Power Dynamics PDI-09S-5 (DE9 male, right-angle THT, 5.0 mm footprint: near pin row 4.94 mm from the board edge, 2 x 3.2 mm holes on 25.0 mm centres; 7.2 mm / 0.318 in parts do NOT fit) - hand-solder, not JLC-assembled"
+			(at 74.93 434.34 0)
+			(hide yes)
+			(effects
+				(font
+					(size 1.27 1.27)
+				)
+			)
+		)
 		(pin "1"
 		)
@@
 			)
 		)
+		(property "Sourcing" "Power Dynamics PDI-09S-5 (DE9 male, right-angle THT, 5.0 mm footprint: near pin row 4.94 mm from the board edge, 2 x 3.2 mm holes on 25.0 mm centres; 7.2 mm / 0.318 in parts do NOT fit) - hand-solder, not JLC-assembled"
+			(at 74.93 504.19 0)
+			(hide yes)
+			(effects
+				(font
+					(size 1.27 1.27)
+				)
+			)
+		)
 		(pin "1"
 		)
@@
 			)
 		)
+		(property "Sourcing" "generic 2.54 mm pin header, 1x6 vertical - hand-solder, not JLC-assembled"
+			(at 320.04 59.69 0)
+			(hide yes)
+			(effects
+				(font
+					(size 1.27 1.27)
+				)
+			)
+		)
 		(pin "1"
 		)
@@
 			)
 		)
+		(property "Sourcing" "generic 2.54 mm pin header, 1x4 vertical - hand-solder, not JLC-assembled"
+			(at 320.04 105.41 0)
+			(hide yes)
+			(effects
+				(font
+					(size 1.27 1.27)
+				)
+			)
+		)
 		(pin "1"
 		)
@@
 			)
 		)
+		(property "Sourcing" "generic 2.54 mm pin header, 1x3 vertical - hand-solder, not JLC-assembled"
+			(at 320.04 143.51 0)
+			(hide yes)
+			(effects
+				(font
+					(size 1.27 1.27)
+				)
+			)
+		)
 		(pin "1"
 		)
@@
 			)
 		)
+		(property "Sourcing" "none - solder bridge, no part to buy"
+			(at 393.7 168.91 0)
+			(hide yes)
+			(effects
+				(font
+					(size 1.27 1.27)
+				)
+			)
+		)
 		(pin "1"
 		)
@@
 			)
 		)
-		(property "LCSC" "TBD:MF-MSMF series"
+		(property "LCSC" "C84140"
 			(at 314.96 264.16 0)
 			(hide yes)
@@
 			)
 		)
-		(property "LCSC" "TBD:MF-MSMF series"
+		(property "LCSC" "C17313"
 			(at 391.16 264.16 0)
 			(hide yes)
@@
 			)
 		)
-		(property "LCSC" "TBD:MF-MSMF series"
+		(property "LCSC" "C17313"
 			(at 419.1 264.16 0)
 			(hide yes)
@@
 			)
 		)
-		(property "LCSC" "TBD:220uF/16V SMD alu"
+		(property "LCSC" "C128533"
+			(at 314.96 320.04 0)
+			(hide yes)
+			(effects
+				(font
+					(size 1.27 1.27)
+				)
+			)
+		)
+		(property "MPN" "EEE-FK1C221XP"
 			(at 314.96 320.04 0)
 			(hide yes)
@@
 			)
 		)
-		(property "LCSC" "TBD:150uF/16V SMD alu"
+		(property "LCSC" "C413656"
+			(at 391.16 320.04 0)
+			(hide yes)
+			(effects
+				(font
+					(size 1.27 1.27)
+				)
+			)
+		)
+		(property "MPN" "EEE-FKC151XAP"
 			(at 391.16 320.04 0)
 			(hide yes)
@@
 			)
 		)
+		(property "Sourcing" "Molex 67643-3910 (USB-A receptacle, right-angle THT; 67643-0910 is the same land) - hand-solder, not JLC-assembled"
+			(at 320.04 424.18 0)
+			(hide yes)
+			(effects
+				(font
+					(size 1.27 1.27)
+				)
+			)
+		)
 		(pin "1"
 		)
@@
 			(at 320.04 490.22 0)
 			(hide yes)
+			(effects
+				(font
+					(size 1.27 1.27)
+				)
+			)
+		)
+		(property "Sourcing" "GCT USB4135-GF-A (USB-C 6P power-only receptacle, top-mount horizontal) - hand-solder, not JLC-assembled"
+			(at 320.04 490.22 0)
+			(hide yes)
