File: kicad/rev6/amigahid-pico-rev6.kicad_sch (KiCad schematic)
At the start: 115 parts, among them J1 A500 KBD OUT, J10 PS/2 KBD OUT, J11 DIN5 KBD IN, J12 PS/2 KBD IN, J13 USB-C AUX 5V, J2 DEBUG UART+SWD, J3 OLED I2C, J4 USB-A HOST, J7 SPARE GP28, J8 A500 KBD IN, J9 DIN5 KBD OUT, P1 DE9 MALE PORT 1, P2 DE9 MALE PORT 2, Q1 BSS138, Q10 BSS138, Q11 BSS138, Q12 BSS138, Q13 BSS138, Q14 BSS138, Q15 BSS138, Q16 BSS138, Q17 BSS138, Q18 BSS138, Q19 BSS138, Q2 BSS138, Q3 BSS138, Q4 BSS138, Q5 BSS138, Q6 BSS138, Q7 BSS138, Q8 BSS138, Q9 BSS138, U1 PicoW, U2 USBLC6-2SC6

Commit message: kicad: mount the oled on a socket and two posts
the 0.96in ssd1306 module now plugs straight down onto the board instead of
hanging off wires: J3 becomes a 1x4 female socket at the module's header edge
(pins x 81.74-89.36, y 40.5) and two M2 posts hold the east edge, H1 (97.3,
40.5) and H2 (97.3, 64.3), 2.2 mm NPTH, board-only footprints.  the module
sits at x 71.8-99.3, y 38.5-66.3, flush inside the east edge.  the other two
corners get no post on purpose: the lower-left one lands on Q18 and six
port-2 nets, the upper-left one sits in the corridor the i2c pair crosses.

  * J3's pin order is the module's, GND VCC SCL SDA, so pins 1 and 2 swap
    nets in the schematic (was 3V3 GND SCL SDA); footprint and Sourcing
    field follow.  a VCC-GND module wants the two labels swapped back.
  * the i2c pair leaves the pico through the lane the redundant +3V3 F.Cu
    loop occupied (the pocket's pull-ups and J7 are fed from the west, via a
    via at the old J3 pad-1 spot and one link down to the pico-side +3V3),
    then 45 mm east to the socket.  /swclk, /swdio and /cont1_b2_lo, which
    ran through the new pad row, are re-threaded north of it.  three GND
    stitch vias re-link pour patches the new lanes walled off.
  * the credit block moves to the bottom silkscreen (the module covers its
    old spot); "AUX 5V" shifts north clear of the module edge.
  * check_rev6_netlist.py: J3 map RE-TARGETED to the socket's pin order
    (1 = gnd, 2 = 3v3); 357/357, nothing relaxed.  check_rev6_pcb.py pins
    the new blob; the commit hash is pinned in the follow-up.
  * doc/errata.md, the mouser bom and the order list carry the mount:
    post length = socket body + 2.54 mm (11 mm for an 8.5 mm socket), never
    under 8 mm because the pico's micro-usb cable passes under the module's
    west edge.

gates: erc 0; drc 0 violations / 0 unconnected / 0 parity; check_rev6_netlist.py
357/357; check_rev6_style.py S1 99.8%, S2 0 staircases, S3 clean;
check_rev6_pcb.py 37/38 - J3 red only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
Parts:
- J3: footprint Connector_PinHeader_2.54mm:PinHeader_1x04_P2.54mm_Vertical -> Connector_PinSocket_2.54mm:PinSocket_1x04_P2.54mm_Vertical; Sourcing generic 2.54 mm pin header, 1x4 vertical - hand-solder, not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 -> generic 2.54 mm female pin socket, 1x4 vertical, TALL body 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
Connections:
- net +3V3: now also J3.2 (Pin_2); no longer J3.1 (Pin_1)
- net GND: now also J3.1 (Pin_1); no longer J3.2 (Pin_2)
Changed lines of the file:
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@@
 			)
 		)
-		(property "Footprint" "Connector_PinHeader_2.54mm:PinHeader_1x04_P2.54mm_Vertical"
+		(property "Footprint" "Connector_PinSocket_2.54mm:PinSocket_1x04_P2.54mm_Vertical"
 			(at 320.04 105.41 0)
 			(hide yes)
@@
 			)
 		)
-		(property "Sourcing" "generic 2.54 mm pin header, 1x4 vertical - hand-solder, not JLC-assembled"
+		(property "Sourcing" "generic 2.54 mm female pin socket, 1x4 vertical, TALL body (8.5 mm standard) - the 0.96in OLED module plugs straight in; hand-solder, not JLC-assembled"
 			(at 320.04 105.41 0)
 			(hide yes)
@@
 		)
 	)
-	(label "+3V3"
+	(label "GND"
 		(at 307.34 102.87 180)
 		(effects
@@
 		)
 	)
-	(label "GND"
+	(label "+3V3"
 		(at 307.34 105.41 180)
 		(effects
